File: sheets/mainboard-common.kicad_sch (KiCad schematic)
At the start: 45 parts, among them J1 Conn_01x04, J2 USB4105, J3 Conn_01x04, J4 Conn_01x16_Socket, J5 Conn_01x16_Socket, J6 Conn_01x16_Socket, J7 Conn_01x16_Socket, U4 AP22916, U5 AP22916

Commit message: More cleanup
Parts:
- removed A2: PowerFeather, PowerFeather:PowerFeather, symbol PowerFeather:PowerFeather
- added A1: PowerFeather_Mainboard, PowerFeather_KiCAD_Lib:PowerFeather_Mainboard, symbol PowerFeather_KiCAD_Lib:PowerFeather_Mainboard
- TP1: value TestPoint -> GND_TP
- TP3, TP4: value TestPoint -> USB_DP_TP
- TP5: value TestPoint -> VBUS_TP
- TP6: value TestPoint -> 3V3P_TP
- TP7: value TestPoint -> BTN_TP
- TP8: value TestPoint -> LED_TP
Connections:
- net USBDM is gone; now on net USB_DP: J2.A7 (D-), J2.B7 (D-), TP3.1
- net USBDP is gone; now on net USB_DM: J2.A6 (D+), J2.B6 (D+), TP4.1
- net +3.3V: now also A1.2 (3V3)
- net +VSW: now also A1.28 (VBAT)
- net A0: now also A1.5 (A0)
- net A1: now also A1.6 (A1)
- net A2: now also A1.7 (A2)
- net A3: now also A1.8 (A3)
- net A4: now also A1.9 (A4)
- net A5: now also A1.10 (A5)
- net D10: now also A1.22 (D10)
- net D11: now also A1.23 (D11)
- net D12: now also A1.24 (D12)
- net D13: now also A1.25 (D13)
- net D2: now also A1.16 (TXD0/D2)
- net D5: now also A1.19 (D5)
- net D6: now also A1.20 (D6)
- net D7: now also A1.31 (D7)
- net D8: now also A1.32 (D8)
- net D9: now also A1.21 (D9)
- net EN: now also A1.27 (EN); no longer R23.2
- net GND: now also A1.29 (GND), A1.4 (GND)
- net MISO: now also A1.13 (MISO)
- net MOSI: now also A1.12 (MOSI)
- net QON: now also A1.3 (QON)
- net RST: now also A1.1 (~{RST}); no longer BTN1.1, C19.2, R15.1
- net RX: now also A1.14 (RX/D0)
- net SCK: now also A1.11 (SCK)
- net SCL: now also A1.18 (SCL)
- net SDA: now also A1.17 (SDA)
- net TX: now also A1.15 (TX/D1)
- net VDC: now also A1.30 (VDC)
- net VS: now also A1.26 (VS)
- net VSQT renamed VCC
- new net: BTN1.1, C19.2, R15.1
- new net EN0: R23.2
Other:
- note added: "Reset"
- note added: "User Button"
- note added: "User LED"
- note added: "Wing Enable"
- moved on the sheet: BTN1, BTN2, C13, C14, C15, C16, C19, C21, C22, C23, C24, C25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
