File: sheets/tps631011.kicad_sch (KiCad schematic)
At the start: 4 parts, among them U2 XC6220B331ER-G

Commit message: More cleanup
Parts:
- removed C11: 1uF, Capacitor_SMD:C_0402_1005Metric, symbol Device:C
- removed U2: XC6220B331ER-G, PowerFeather:USP-6C_TOR, symbol Regulator_Linear:XC6220B331MR
- added L2: L, symbol Device:L
- added R6, R7: R_US, symbol Device:R_US
- added U2: TPS631011, symbol PowerFeather_KiCAD_Lib:TPS631011
- C2: value 10uF -> C; footprint Capacitor_SMD:C_0603_1608Metric -> (none); Comment 10V, X5R -> (none); MPN 187-CL10A106KP8NNWC -> (none)
- C8: value 4.7uF -> C; footprint Capacitor_SMD:C_0603_1608Metric -> (none); Comment 10V, X5R -> (none); MPN 187-CL10A475KP8NNND -> (none)
Connections:
- net GND: now also C2.2, R7.2, U2.B2 (MODE), U2.C2 (GND); no longer C2.1
- net VIN: now also C8.1, U2.A1 (VIN), U2.A2 (EN); no longer C2.2
- net VOUT: now also C2.1, R6.1, U2.D1 (VOUT); no longer C8.1
- new net: R6.2, R7.1, U2.D2 (FB)
- new net: L2.1, U2.B1 (L1)
- new net: L2.2, U2.C1 (L2)

Commit message: More cleanup
Parts:
- renumbered C8 to C20, C2 to C21, R6 to R18, R7 to R19, U2 to U5
Changed lines of the file:
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@@
 		(dnp no)
 		(fields_autoplaced yes)
-		(property "Reference" "C8"
+		(property "Reference" "C20"
 			(at 77.47 67.3099 0)
 			(effects
@@
 		(instances
 			(project "esp32s3-powerfeather"
-				(path "/5be6a852-fa78-49fa-bb8c-8d5ad39f4b26/46173bec-ea31-4af7-a417-264e4953a5cb/1c9cf99d-29d3-45e3-bf18-d4466a37473a"
-					(reference "C8")
+				(path "/5be6a852-fa78-49fa-bb8c-8d5ad39f4b26/a940761a-0d45-4491-ba89-ec093a8f239f/1c9cf99d-29d3-45e3-bf18-d4466a37473a"
+					(reference "C20")
 					(unit 1)
 				)
@@
 		(dnp no)
 		(fields_autoplaced yes)
-		(property "Reference" "C2"
+		(property "Reference" "C21"
 			(at 140.97 66.0399 0)
 			(effects
@@
 		)
 		(instances
-			(project ""
-				(path "/5be6a852-fa78-49fa-bb8c-8d5ad39f4b26/46173bec-ea31-4af7-a417-264e4953a5cb/1c9cf99d-29d3-45e3-bf18-d4466a37473a"
-					(reference "C2")
+			(project "esp32s3-powerfeather"
+				(path "/5be6a852-fa78-49fa-bb8c-8d5ad39f4b26/a940761a-0d45-4491-ba89-ec093a8f239f/1c9cf99d-29d3-45e3-bf18-d4466a37473a"
+					(reference "C21")
 					(unit 1)
 				)
@@
 		(dnp no)
 		(fields_autoplaced yes)
-		(property "Reference" "R7"
+		(property "Reference" "R19"
 			(at 127 71.1199 0)
 			(effects
@@
 		(instances
 			(project "esp32s3-powerfeather"
-				(path "/5be6a852-fa78-49fa-bb8c-8d5ad39f4b26/46173bec-ea31-4af7-a417-264e4953a5cb/1c9cf99d-29d3-45e3-bf18-d4466a37473a"
-					(reference "R7")
+				(path "/5be6a852-fa78-49fa-bb8c-8d5ad39f4b26/a940761a-0d45-4491-ba89-ec093a8f239f/1c9cf99d-29d3-45e3-bf18-d4466a37473a"
+					(reference "R19")
 					(unit 1)
 				)
@@
 		(dnp no)
 		(fields_autoplaced yes)
-		(property "Reference" "U2"
+		(property "Reference" "U5"
 			(at 106.68 48.26 0)
 			(effects
@@
 		)
 		(instances
-			(project ""
-				(path "/5be6a852-fa78-49fa-bb8c-8d5ad39f4b26/46173bec-ea31-4af7-a417-264e4953a5cb/1c9cf99d-29d3-45e3-bf18-d4466a37473a"
-					(reference "U2")
+			(project "esp32s3-powerfeather"
+				(path "/5be6a852-fa78-49fa-bb8c-8d5ad39f4b26/a940761a-0d45-4491-ba89-ec093a8f239f/1c9cf99d-29d3-45e3-bf18-d4466a37473a"
+					(reference "U5")
 					(unit 1)
 				)
@@
 		)
 		(instances
-			(project ""
-				(path "/5be6a852-fa78-49fa-bb8c-8d5ad39f4b26/46173bec-ea31-4af7-a417-264e4953a5cb/1c9cf99d-29d3-45e3-bf18-d4466a37473a"
+			(project "esp32s3-powerfeather"
+				(path "/5be6a852-fa78-49fa-bb8c-8d5ad39f4b26/a940761a-0d45-4491-ba89-ec093a8f239f/1c9cf99d-29d3-45e3-bf18-d4466a37473a"
 					(reference "L2")
 					(unit 1)
@@
 		(dnp no)
 		(fields_autoplaced yes)
-		(property "Reference" "R6"
+		(property "Reference" "R18"
 			(at 127 60.9599 0)
 			(effects
@@
 		)
 		(instances
-			(project ""
-				(path "/5be6a852-fa78-49fa-bb8c-8d5ad39f4b26/46173bec-ea31-4af7-a417-264e4953a5cb/1c9cf99d-29d3-45e3-bf18-d4466a37473a"
-					(reference "R6")
-					(unit 1)
-				)
+			(project "esp32s3-powerfeather"
+				(path "/5be6a852-fa78-49fa-bb8c-8d5ad39f4b26/a940761a-0d45-4491-ba89-ec093a8f239f/1c9cf99d-29d3-45e3-bf18-d4466a37473a"
+					(reference "R18")
+					(unit 1)
+				)
