File: sheets/bq25622e.kicad_sch (KiCad schematic)
At the start: 15 parts, among them U6 BQ25622E

Commit message: Fill in missing component details
Parts:
- LED2: value C190KRKT -> LTST-C190KRKT
- U6: MPN (none) -> 595-BQ25622ERYKR
Changed lines of the file:
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@@
 			)
 		)
-		(property "Value" "C190KRKT"
+		(property "Value" "LTST-C190KRKT"
 			(at 60.96 44.704 0)
 			(effects
@@
 			(at 102.87 63.5 0)
 			(effects
+				(font
+					(size 1.27 1.27)
+				)
+				(hide yes)
+			)
+		)
+		(property "MPN" "595-BQ25622ERYKR"
+			(at 102.87 63.5 0)
+			(effects

Commit message: Fix pcb import warnings
Parts:
- U6: MPN 595-BQ25622ERYKR -> 595-BQ25622RYKR
Changed lines of the file:
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@@
+	)
+	(symbol
+		(lib_id "PowerFeather_KiCAD_Lib:BQ25622E")
+		(at 102.87 63.5 0)
+		(unit 1)
+		(exclude_from_sim no)
+		(in_bom yes)
+		(on_board yes)
+		(dnp no)
+		(fields_autoplaced yes)
+		(property "Reference" "U6"
+			(at 102.87 40.64 0)
+			(effects
+				(font
+					(size 1.27 1.27)
+				)
+			)
+		)
+		(property "Value" "BQ25622E"
+			(at 102.87 43.18 0)
+			(effects
+				(font
+					(size 1.27 1.27)
+				)
+			)
+		)
+		(property "Footprint" "PowerFeather_KiCAD_Lib:BQ25622E"
+			(at 102.108 83.312 0)
+			(effects
+				(font
+					(size 1.27 1.27)
+				)
+				(hide yes)
+			)
+		)
+		(property "Datasheet" "https://www.ti.com/lit/gpn/bq25622e"
+			(at 104.14 85.344 0)
+			(effects
+				(font
+					(size 1.27 1.27)
+				)
+				(hide yes)
+			)
+		)
+		(property "Description" "BQ25622E I2C Controlled 1-Cell, 3A, Maximum 18V Input, Buck Battery Charger with NVDC Power Path Management"
+			(at 102.87 63.5 0)
+			(effects
+				(font
+					(size 1.27 1.27)
+				)
+				(hide yes)
+			)
+		)
+		(property "MPN" "595-BQ25622RYKR"
+			(at 102.87 63.5 0)
+			(effects
+				(font
+					(size 1.27 1.27)
+				)
+				(hide yes)
+			)
+		)
+		(pin "9"
+		)
+		(pin "5"
+		)
+		(pin "4"
+		)
+		(pin "16"
+		)
+		(pin "12"
+		)
+		(pin "17"
+		)
+		(pin "6"
+		)
+		(pin "3"
+		)
+		(pin "10"
+		)
+		(pin "14"
+		)
+		(pin "2"
+		)
+		(pin "7"
+		)
+		(pin "11"
+		)
+		(pin "15"
+		)
+		(pin "8"
+		)
+		(pin "18"
+		)
+		(pin "13"
+		)
+		(pin "1"
+		)
+		(instances
+			(project ""
+				(path "/351775ff-22dd-4601-a146-0ae5bb7b1807/788c158d-fb18-46fd-a4f8-fb3433f7b73b"
+					(reference "U6")
+					(unit 1)
+				)
+			)
+		)
 	)
 	(symbol
@@
 					(unit 1)
 				)
-			)
-		)
-	)
-	(symbol
-		(lib_id "PowerFeather_KiCAD_Lib:BQ25622E")
-		(at 102.87 63.5 0)
-		(unit 1)
-		(exclude_from_sim no)
-		(in_bom yes)
-		(on_board yes)
-		(dnp no)
-		(fields_autoplaced yes)
-		(property "Reference" "U6"
-			(at 102.87 40.64 0)
-			(effects
-				(font
-					(size 1.27 1.27)
-				)
-			)
-		)
-		(property "Value" "BQ25622E"
-			(at 102.87 43.18 0)
-			(effects
-				(font
-					(size 1.27 1.27)
-				)
-			)
-		)
-		(property "Footprint" "PowerFeather_KiCAD_Lib:BQ25622E"
-			(at 102.108 83.312 0)
-			(effects
-				(font
-					(size 1.27 1.27)
-				)
-				(hide yes)
-			)
-		)
-		(property "Datasheet" "https://www.mouser.com/datasheet/2/405/1/bq25628e-3377636.pdf"
-			(at 104.14 85.344 0)
-			(effects
-				(font
-					(size 1.27 1.27)
-				)
-				(hide yes)
-			)
-		)
-		(property "Description" ""
-			(at 102.87 63.5 0)
-			(effects
-				(font
-					(size 1.27 1.27)
-				)
-				(hide yes)
-			)
-		)
-		(property "MPN" "595-BQ25622ERYKR"
-			(at 102.87 63.5 0)
-			(effects
-				(font
-					(size 1.27 1.27)
-				)
-				(hide yes)
-			)
-		)
-		(pin "5"
-		)
-		(pin "15"
-		)
-		(pin "3"
-		)
-		(pin "17"
-		)
-		(pin "13"
-		)
-		(pin "10"
-		)
-		(pin "12"
-		)
-		(pin "1"
-		)
-		(pin "11"
-		)
-		(pin "14"
-		)
-		(pin "18"
-		)
-		(pin "16"
-		)
-		(pin "7"
-		)
-		(pin "2"
-		)
-		(pin "8"
-		)
-		(pin "4"
-		)
-		(pin "6"
-		)
-		(pin "9"
-		)
-		(instances
-			(project ""
-				(path "/351775ff-22dd-4601-a146-0ae5bb7b1807/788c158d-fb18-46fd-a4f8-fb3433f7b73b"
-					(reference "U6")
-					(unit 1)
-				)

Commit message: Change out values of some parts
- Fix max17260 sku
- Use 800 ohms for stat pin
- Change charger inductor value
Parts:
- L2: MPN 81-DFE252012P-1R0MP2 -> 815-AOTB252010S1R0MT
- R26, R28: MPN 603-RT0402BRD075K36L -> 603-RC0402FR-135K36L
- R27: value 1.2k -> 800; MPN 603-AC0402FR-07845RL -> 603-RC0402FR-7W806RL
- R29: MPN 603-RT0402BRD0731K6L -> 603-RC0402FR-7D31K6L
Changed lines of the file:
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@@
 			)
 		)
-		(property "Value" "1.2k"
+		(property "Value" "800"
 			(at 84.074 60.198 90)
 			(effects
@@
 			)
 		)
-		(property "Datasheet" "https://www.mouser.ph/datasheet/2/447/PYu_AC_51_RoHS_L_9-3005297.pdf"
+		(property "Datasheet" "https://www.mouser.com/datasheet/2/447/PYu_RC_Group_51_RoHS_L_11-1984063.pdf"
 			(at 77.47 58.42 0)
 			(effects
@@
 			)
 		)
-		(property "MPN" "603-AC0402FR-07845RL"
+		(property "MPN" "603-RC0402FR-7W806RL "
 			(at 77.47 58.42 0)
 			(effects
@@
 			)
 		)
-		(property "Datasheet" "https://www.mouser.jp/datasheet/2/281/1/J_E_TE243A_0032-2303193.pdf"
+		(property "Datasheet" "https://www.mouser.com/datasheet/2/3/AOTA_B252010S-3224149.pdf"
 			(at 135.89 53.34 0)
 			(effects
@@
 			)
 		)
-		(property "MPN" "81-DFE252012P-1R0MP2"
+		(property "MPN" "815-AOTB252010S1R0MT"
 			(at 135.89 53.34 0)
 			(effects
@@
 			)
 		)
-		(property "Datasheet" "https://www.mouser.ph/datasheet/2/447/PYu_RT_1_to_0_01_RoHS_L_12-3003070.pdf"
+		(property "Datasheet" "https://www.mouser.com/datasheet/2/447/PYu_RC_Group_51_RoHS_L_12-3368608.pdf"
 			(at 72.39 46.99 0)
 			(effects
@@
 			)
 		)
-		(property "MPN" "603-RT0402BRD075K36L"
+		(property "MPN" "603-RC0402FR-135K36L"
 			(at 72.39 46.99 0)
 			(effects
@@
 			)
 		)
-		(property "Datasheet" "https://www.mouser.ph/datasheet/2/447/PYu_RT_1_to_0_01_RoHS_L_12-3003070.pdf"
+		(property "Datasheet" "https://www.mouser.com/datasheet/2/447/PYu_RC_Group_51_RoHS_L_12-3368608.pdf"
 			(at 127 73.66 0)
 			(effects
@@
 			)
 		)
-		(property "MPN" "603-RT0402BRD075K36L"
+		(property "MPN" "603-RC0402FR-135K36L"
 			(at 127 73.66 0)
 			(effects
@@
 			)
 		)
-		(property "Datasheet" "https://www.mouser.ph/datasheet/2/447/PYu_RT_1_to_0_01_RoHS_L_12-3003070.pdf"
+		(property "Datasheet" "https://www.mouser.com/datasheet/2/447/PYu_RC_Group_51_RoHS_L_11-1984063.pdf"
 			(at 127 85.09 0)
 			(effects
@@
 			)
 		)
-		(property "MPN" "603-RT0402BRD0731K6L"
+		(property "MPN" "603-RC0402FR-7D31K6L"
 			(at 127 85.09 0)
 			(effects
